File: saha-cpu.sch (EAGLE design)
At the start: 47 parts, among them X2 X3815-10, X3 S4B-PH-SM4-TB

Commit message: schematic update
Parts:
- added C21, C23, C24, C25, C26, C27: 100n 0603, saha-cpu:CAP0603
- added C22: (no value), saha-cpu:CAP0603
- added C28, C29, C30: 4u7 0805, saha-cpu:CAP0805
- added D5: 74AHC14, saha-cpu:74AHC14
- added H1, H2: LED-GRN, saha-cpu:LED-GRN
- added H3: LED-RED, saha-cpu:LED-RED
- added L5: BLM31KN601, saha-cpu:IND1206
- added L6: NRS4018-4U7, saha-cpu:NRS4018-4U7
- added R12, R13, R14, R16, R17, R18, R19, R20, R21: (no value), saha-cpu:RES0603
- added R15: 10k0, saha-cpu:RES0603
- added R22, R25, R27, R29: 499R 0805, saha-cpu:RES0805
- added R23, R24, R26, R28: 33k2, saha-cpu:RES0603
- added R30: 1, saha-cpu:RES2512
- added X4, X5: S4B-PH-SM4-TB, saha-cpu:S4B-PH-SM4-TB
- added X6: S8B-PH-SM4-TB, saha-cpu:S8B-PH-SM4-TB
- added Y1, Y2, Y3, Y4: PTH-ROUND3.2-6.5ROUND, saha-cpu:PTH-ROUND3.2-6.5ROUND
- R8, R9: value 2k2 -> 10k0
- V1: value SMAJXXA -> SMAJ15A
Connections:
- net N$10 renamed SWCLK
- net N$11 renamed SWDIO-CPU
- net N$12 renamed SWCLK-CPU
- net N$13 renamed VCAP
- net N$14 renamed VDDA
- net N$15 renamed SDA
- net N$16 renamed SCL
- net N$17 renamed D5V
- net N$6 renamed OSCOUT
- net N$8 renamed OSCIN
- net N$9 renamed SWDIO
- new net DIR1: R17.2, X4.3
- new net DIR2: R19.2, X5.3
- new net DIR_1: D2G$2.PA4, D3.A2
- new net DIR_2: D2G$2.PA5, D3.A4
- new net IN1: R22.1, R23.1, X6.1
- new net IN1_F: C24.1, D5G$1.A, R23.2
- new net IN2: R24.1, R25.1, X6.3
- new net IN2_F: C25.1, D5G$2.A, R24.2
- new net IN3: R26.1, R27.1, X6.5
- new net IN3_F: C26.1, D5G$3.A, R26.2
- new net IN4: R28.1, R29.1, X6.7
- new net IN4_F: C27.1, D5G$4.A, R28.2
- new net IN_1: D2G$2.PC10, D5G$1.Y
- new net IN_2: D2G$2.PC11, D5G$2.Y
- new net IN_3: D2G$2.PC12, D5G$3.Y
- new net IN_4: D2G$2.PB11, D5G$4.Y
- new net LEDGRN: D2G$2.PC8, H2.A
- new net LEDRED: D2G$2.PC9, H3.A
- new net MEAS_VBAT: C22.1, D2G$1.PA0/WKUP, R20.2, R21.1
- new net N$21: D3.Y4, R19.1
- new net N$22: H1.C, R12.2
- new net N$23: H3.C, R13.2
- new net N$24: H2.C, R14.2
- new net N$25: D3.Y3, R18.1
- new net N$26: D3.Y2, R17.1
- new net N$27: D3.Y1, R16.1
- new net N$6: C28.1, L5.2, R30.2, V1.C
- new net N$8: R30.1, X1.1
- new net N$9: C29.1, L5.1, L6.2
- new net OE_N: D2G$2.PA1, D3.OE1, D3.OE2, D3.OE3, D3.OE4, R15.1
- new net PULSE1: R16.2, X4.1
- new net PULSE2: R18.2, X5.1
- new net PULSE_1: D2G$2.PA2, D3.A1
- new net PULSE_2: D2G$2.PA3, D3.A3
- net +3V3: now also C23.1, D5G$1.VCC, H1.A, R15.2
- net +5V: now also C21.1, D3.VCC, R22.2, R25.2, R27.2, R29.2
- net +VBAT: now also C30.1, L6.1, R21.2; no longer V1.C, X1.1
- net GND: now also C21.2, C22.2, C23.2, C24.2, C25.2, C26.2, C27.2, C28.2, C29.2, C30.2, D3.GND, D5G$1.GND, D5G$5.A, D5G$6.A, R12.1, R13.1, R14.1, R20.1, X4.2, X4.4, X5.2, X5.4, X6.2, X6.4, X6.6, X6.8, Y1.1, Y2.1, Y3.1, Y4.1
Other:
- note added: "ADC1_0"
- note added: "TIM9_CH1"
- note added: "TIM9_CH2"

Commit message: Initial routing complete
Parts:
- added C31: 4u7 0805, saha-cpu:CAP0805
- added C32, C33: 22u 0805, saha-cpu:CAP0805
Connections:
- net N$2 renamed SW3V3
- net N$4 renamed SW5V
- net N$6 renamed VINR
- net N$8 renamed VIN
- net N$9 renamed VINL
- removed net N$18: C18.2, X3.3
- net +3V3: now also C33.1
- net +5V: now also C32.1
- net +VBAT: now also C31.1
- net GND: now also C18.2, C31.2, C32.2, C33.2, X3.3
- net MEAS_VBAT: now also D2G$2.PA7; no longer D2G$1.PA0/WKUP
Other:
- note added: "ADC1_7"
- note removed: "ADC1_0"
- moved on the sheet: C22, R20, R21
