File: saha-cpu.brd (EAGLE design)
At the start: 100 x 56 mm, 89 parts, among them X2 X3815-10, X3 S4B-PH-SM4-TB, X4 S4B-PH-SM4-TB, X5 S4B-PH-SM4-TB, X6 S8B-PH-SM4-TB, Y1 PTH-ROUND3.2-6.5ROUND, Y2 PTH-ROUND3.2-6.5ROUND, Y3 PTH-ROUND3.2-6.5ROUND, Y4 PTH-ROUND3.2-6.5ROUND

Commit message: Initial routing complete
Parts:
- added C31: 4u7 0805, saha-cpu:C0805
- added C32, C33: 22u 0805, saha-cpu:C0805
- moved R21 38.1 mm to (20.4, 16.6), turned to 180 degrees
- moved R20 37.1 mm to (23.4, 16.6), turned to 180 degrees
- moved D1 24.9 mm to (50.3, 8.20), turned to 180 degrees
- moved R5 23.9 mm to (52.8, 8.50), turned to 270 degrees
- moved C7 23.0 mm to (47.8, 8.50), turned to 90 degrees
- moved R7 13.9 mm to (78.1, 21.4), turned to 180 degrees
- moved C17 9.57 mm to (78.1, 19.2), turned to 0 degrees
- moved C22 8.28 mm to (68.6, 6.20), turned to 270 degrees
- moved C14 7.80 mm to (74.5, 8.07), turned to 270 degrees
- moved C16 7.32 mm to (64.5, 24.2)
- moved C15 6.40 mm to (65.4, 6.87), turned to 180 degrees
- moved R6 5.64 mm to (78.1, 17.5), turned to 180 degrees
- moved R15 5.42 mm to (35.1, 32.5)
- moved C21 3.51 mm to (28.1, 30.4)
- moved R13 3.00 mm to (89.4, 18.0)
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Connections:
- net N$2 renamed SW3V3
- net N$4 renamed SW5V
- net N$6 renamed VINR
- net N$8 renamed VIN
- net N$9 renamed VINL
- removed net N$18: C18.2, X3.3
- net +3V3: now also C33.1
- net +5V: now also C32.1
- net +VBAT: now also C31.1
- net GND: now also C18.2, C31.2, C32.2, C33.2, X3.3
- net MEAS_VBAT: now also D2.23; no longer D2.14
Routing:
- net +3V3: track 0.00 -> 237.9 mm, vias 0 -> 13
- net +5V: track 0.00 -> 147.4 mm, vias 0 -> 12
- net OE_N: track 0.00 -> 99.8 mm
- net GND: track 0.00 -> 95.7 mm, vias 0 -> 148
- net DIR_1: track 0.00 -> 74.4 mm
- net DIR_2: track 0.00 -> 73.5 mm
- net PULSE_2: track 0.00 -> 72.5 mm
- net RESET_N: track 0.00 -> 71.5 mm
- net MEAS_VBAT: track 0.00 -> 66.4 mm
- net PULSE_1: track 0.00 -> 65.2 mm
- net +VBAT: track 0.00 -> 47.0 mm
- net I2C1SCL: track 0.00 -> 38.5 mm
- net I2C1SDA: track 0.00 -> 36.4 mm
- net USART6RX: track 0.00 -> 29.5 mm
- net USART6TX: track 0.00 -> 28.6 mm
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- added copper zone on layer 1, net +3V3
- added copper zone on layer 1, net +5V
- added copper zone on layer 1, net +VBAT
- added copper zone on layer 1, net GND
- added copper zone on layer 16, net GND
- added copper zone on layer 1, net SW3V3
- added copper zone on layer 1, net SW5V
- added copper zone on layer 1, net VIN
- added copper zone on layer 1, net VINL
- added copper zone on layer 1, net VINR
Other:
- board text added: "ERR"
- board text added: "PWR"
- board text added: "RUN"

Commit message: routing finished
Parts:
- moved U$1 20.0 mm to (22.6, 10.7)
Routing:
- net GND: vias 148 -> 147
- added copper zone on layer 16, net N$2
- added copper zone on layer 1, net N$4
Other:
- board text added: "+"
- board text added: "+5V SDA GND SCL"
- board text added: "-"
- board text added: "1"
- board text added: "2"
- board text added: "IN1 GND IN2 GND IN3 GND IN4 GND"
- board text added: "KIMMOLI 2019"
- board text added: "PULSE1 GND DIR1 GND"
- board text added: "PULSE2 GND DIR2 GND"
- board text added: "SAHA CPU"
- board text added: "V1.0"

Commit message: fine tuning
Parts:
- moved C10 0.90 mm to (56.5, 13.4)
- moved C11 0.90 mm to (56.5, 20.4)
- moved G1 0.90 mm to (56.5, 16.9)
Routing:
- net USART6TX: track 28.6 -> 29.8 mm
- net +3V3: track 237.9 -> 236.7 mm
- net GND: vias 147 -> 164
- removed copper zone on layer 16, net N$2
- removed copper zone on layer 1, net N$4
